File: FlashSd.kicad_sch (KiCad schematic)
At the start: 0 parts

Commit message: began fixing schematic added barometer
Parts:
- added D1: SRV05-4.TCT, myFootprints:SOT95P280X145-6N, symbol SRV05-4.TCT:SRV05-4.TCT
- added J8: Micro_SD_Card, symbol Connector:Micro_SD_Card
- added R18: 10k, symbol Device:R
- added R19: .022k, symbol Device:R
Connections:
- new net: J8.2 (DAT3/CD), R18.2
- new net: J8.5 (CLK), R19.2
- new net +3.3V: D1.5, J8.4 (VDD), R18.1
- new net GND: D1.2, J8.6 (VSS), J8.9 (SHIELD)
- new net SDCLK: R19.1
- new net SDMISO: D1.4, J8.3 (CMD)
- new net SDMOSI: D1.6, J8.7 (DAT0)
- no-connect marks 0 -> 4
