File: Schematics/flightcomputer2.kicad_pcb (KiCad board)
At the start: 4 copper layers, 80 x 80 mm, 86 parts, among them J1 Microsemi_FlashPro-JTAG-10, J2 Pyro, J3 USB_C_Receptacle, J4 Pyro, J5 Conn_01x05_Pin, J6 Conn_01x05_Pin, J7 Conn_Coaxial_Small, J8 Micro_SD_Card, Q1 BSC098N10NS5, Q2 BSC098N10NS5, Q3 BC817, U1 STM32F405RGT6, U2 SN65HVD230, U3 PowerIn, U4 LDL1117-3.3, U5 RFM95W-915S2, U6 MPL3115A2R1, U7 LSM6DS3TR-C, U8 W25Q128JVP, U9 H3LIS100DL, Y1 8mhz

Commit message: layout updated finalizing routing
Parts:
- moved C20 8.83 mm to (163.5, 76.8), turned to 180 degrees
- moved C28 7.99 mm to (151.2, 78.1), turned to 0 degrees
- moved C21 6.02 mm to (163.5, 74.7), turned to 180 degrees
- moved C22 4.71 mm to (160.5, 75.6), turned to -90 degrees
- moved C27 3.80 mm to (151.2, 76.0), turned to 0 degrees
- moved U9 3.44 mm to (151.6, 72.4), turned to 0 degrees
- moved U6 3.02 mm to (161.2, 71.8), turned to 90 degrees
- moved R1 1.61 mm to (127.5, 92.9), turned to 90 degrees
- moved C13 1.04 mm to (154.2, 94.1)
- moved C9 1.04 mm to (154.1, 102.1)
- moved FB1 1.04 mm to (155.1, 99.1)
- moved C10 1.04 mm to (154.2, 96.2)
- moved C14 1.04 mm to (154.2, 92.0)
- moved C15 1.01 mm to (154.5, 85.3)
- moved C16 1.01 mm to (147.7, 87.8)
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Routing:
- net /LoRa/sxMOSI: track 2.91 -> 44.7 mm, vias 1 -> 2
- net /LoRa/sxNSS: track 8.42 -> 46.6 mm, vias 1 -> 2
- net /Accelerometer/AccelerometerSDA: track 3.03 -> 39.8 mm, vias 2 -> 4
- net /Accelerometer/AccelerometerSCL: track 2.04 -> 38.8 mm, vias 1 -> 4
- net /LoRa/sxReset: track 10.6 -> 47.2 mm, vias 1 -> 2
- net /LoRa/sxSCK: track 6.02 -> 42.0 mm, vias 1 -> 2
- net /LoRa/sxMIS0: track 12.4 -> 43.6 mm, vias 1 -> 2
- net /FlashSd/SDMOSI: track 2.33 -> 30.6 mm, vias 1 -> 2
- net /FlashSd/SDMISO: track 2.33 -> 27.6 mm, vias 1 -> 2
- net /LoRa/sxDIO1: track 2.95 -> 26.7 mm, vias 1 -> 2
- net /FlashSd/SDCLK: track 1.40 -> 20.1 mm, vias 1 -> 2
- net +3.3V: track 88.3 -> 106.5 mm, vias 17 -> 20
- net /MCU/D+: track 7.79 -> 25.9 mm
- net /MCU/D-: track 10.2 -> 26.7 mm
- net /MCU/BOOT0: track 8.87 -> 1.94 mm, vias 1 -> 0
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Other:
- board text added: "Boot"
- board text added: "Reset"
- board text added: "Sensors"
