File: Schematics/usb_type_c_sch.kicad_sch (KiCad schematic)
At the start: 4 parts, among them J2 USB_C_Receptacle_USB2.0_16P

Commit message: added final lcsc parts
Parts:
- J2: LCSC Part (none) -> C165948
Changed lines of the file:
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@@
+			)
+		)
+		(property "LCSC Part" "C165948"
+			(at 107.95 72.39 0)
+			(effects
+				(font
+					(size 1.27 1.27)
+				)
+				(hide yes)
 			)
 		)
