File: Schematics/LoRa.kicad_sch (KiCad schematic)
At the start: 2 parts, among them J7 Conn_Coaxial_Small, U5 RFM95W-915S2

Commit message: added comments, awaiting review
Other:
- note added: "Lora module to coaxial connector"
Changed lines of the file:
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@@
 	(generator_version "9.0")
 	(paper "A4")
+	(text "Lora module to coaxial connector"
+		(exclude_from_sim no)
+		(at 134.366 56.388 0)
+		(effects
+			(font
+				(size 1.27 1.27)
+			)
+		)
+	)
 	(junction
 		(at 128.27 100.33)
