File: Schematics/AuxPyro.kicad_sch (KiCad schematic)
At the start: 8 parts, among them J2 Pyro, Q1 IRLML2502TRPBF

Commit message: updated to KiCad 10.0, updated .gitignore
Parts:
- J2: now left out of the parts list
- R21: LCSC C95781 -> C17513
- R24: LCSC C84376 -> C17414
- R26: LCSC C2933415 -> C17713
Changed lines of the file:
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@@
 			)
 		)
-		(property "LCSC" "C2933415"
+		(property "LCSC" "C17713"
 			(at 119.38 100.33 0)
 			(effects
@@
 		(unit 1)
 		(exclude_from_sim no)
-		(in_bom yes)
+		(in_bom no)
 		(on_board yes)
 		(dnp no)
@@
 			)
 		)
-		(property "LCSC" "C95781"
+		(property "LCSC" "C17513"
 			(at 130.81 93.98 90)
 			(effects
@@
 			)
 		)
-		(property "LCSC" "C84376"
-			(at 166.37 95.25 0)
-			(effects
+		(property "LCSC" "C17414"
+			(at 166.37 95.25 0)
+			(effects
