File: Schematics/Can_transceiver.kicad_sch (KiCad schematic)
At the start: 6 parts, among them U2 SN65HVD230

Commit message: updated to KiCad 10.0, updated .gitignore
Parts:
- CAN_IN1, CAN_OUT1: now left out of the parts list
- R8: LCSC C269726 -> C17437
Changed lines of the file:
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@@
 		(unit 1)
 		(exclude_from_sim no)
-		(in_bom yes)
+		(in_bom no)
 		(on_board yes)
 		(dnp no)
@@
 			)
 		)
-		(property "LCSC" "C269726"
+		(property "LCSC" " C17437"
 			(at 156.21 90.17 0)
 			(effects
@@
 		(unit 1)
 		(exclude_from_sim no)
-		(in_bom yes)
+		(in_bom no)
 		(on_board yes)
 		(dnp no)

Commit message: updated stlink
Parts:
- U2: LCSC C1543812 -> C12084
