File: Schematics/GPS1.kicad_sch (KiCad schematic)
At the start: 2 parts, among them J5 Conn_01x05_Pin, J6 Conn_01x05_Pin

Commit message: added comments, awaiting review
Other:
- note added: "External GPS breakout connectors will wire connectors by hand"
- moved on the sheet: J5, J6

Commit message: updated to KiCad 10.0, updated .gitignore
Parts:
- J5, J6: now left out of the parts list
Changed lines of the file:
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@@
 		(unit 1)
 		(exclude_from_sim no)
-		(in_bom yes)
+		(in_bom no)
 		(on_board yes)
 		(dnp no)
@@
 		(unit 1)
 		(exclude_from_sim no)
-		(in_bom yes)
+		(in_bom no)
 		(on_board yes)
 		(dnp no)
