File: Schematics/IMU.kicad_sch (KiCad schematic)
At the start: 4 parts, among them U7 LSM6DS3TR-C

Commit message: reviewed schematic and pcb and replaced part numbers, added and named datasheets into document folder
Parts:
- U7: LCSC C967633 -> C2655100
Changed lines of the file:
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@@
 			)
 		)
-		(property "LCSC" "C967633"
+		(property "LCSC" "C2655100"
 			(at 139.7 113.03 0)
 			(effects

Commit message: updated to KiCad 10.0, updated .gitignore
Parts:
- R36: LCSC C84376 -> C17414
Changed lines of the file:
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@@
 			)
 		)
-		(property "LCSC" "C84376"
+		(property "LCSC" "C17414"
 			(at 121.92 90.17 0)
 			(effects
