File: Schematics/FlashSd.kicad_sch (KiCad schematic)
At the start: 2 parts, among them J8 Micro_SD_Card

Commit message: V2 ready to for order,use prior branches for V1 code
Connections:
- net SDMISO: now also J8.7 (DAT0); no longer J8.3 (CMD)
- net SDMOSI: now also J8.3 (CMD); no longer J8.7 (DAT0)
Changed lines of the file:
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@@
-	(wire
-		(pts
-			(xy 90.17 100.33) (xy 134.62 100.33)
-		)
-		(stroke
-			(width 0)
-			(type default)
-		)
-	)
 	(wire
 		(pts
 			(xy 132.08 97.79) (xy 134.62 97.79)
-		)
-		(stroke
-			(width 0)
-			(type default)
-		)
-	)
-	(wire
-		(pts
-			(xy 90.17 90.17) (xy 134.62 90.17)
 		)
 		(stroke
@@
 	(wire
 		(pts
+			(xy 90.17 100.33) (xy 134.62 100.33)
+		)
+		(stroke
+			(width 0)
+			(type default)
+		)
+	)
+	(wire
+		(pts
 			(xy 132.08 92.71) (xy 134.62 92.71)
+		)
+		(stroke
+			(width 0)
+			(type default)
+		)
+	)
+	(wire
+		(pts
+			(xy 90.17 90.17) (xy 134.62 90.17)
 		)
 		(stroke
@@
 	(hierarchical_label "SDMISO"
 		(shape input)
-		(at 90.17 90.17 180)
+		(at 90.17 100.33 180)
 		(effects
 			(font
@@
 	(hierarchical_label "SDMOSI"
 		(shape input)
-		(at 90.17 100.33 180)
+		(at 90.17 90.17 180)
 		(effects
 			(font
