File: Schematics/MCU.kicad_sch (KiCad schematic)
At the start: 33 parts, among them J3 Conn_ARM_JTAG_SWD_10, Q3 BC817, SW1 SAMZO G4R0015010, SW2 SAMZO G4R0015010, U1 STM32F405RGT6, Y1 8mhz

Commit message: full output submited
Parts:
- J3: LCSC (none) -> C22438120
- R2: LCSC C149504 -> C17414
- R33: LCSC (none) -> C17414
Changed lines of the file:
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@@
 			)
 		)
-		(property "LCSC" "C149504"
+		(property "LCSC" "C17414"
 			(at 40.64 138.43 90)
 			(hide yes)
@@
 			)
 		)
+		(property "LCSC" "C22438120"
+			(at 238.76 52.07 0)
+			(hide yes)
+			(show_name no)
+			(do_not_autoplace no)
+			(effects
+				(font
+					(size 1.27 1.27)
+				)
+			)
+		)
 		(pin "1"
 		)
@@
 			(at 203.2 129.54 0)
 			(hide yes)
+			(show_name no)
+			(do_not_autoplace no)
+			(effects
+				(font
+					(size 1.27 1.27)
+				)
+			)
+		)
+		(property "LCSC" "C17414"
+			(at 203.2 129.54 0)
+			(hide yes)
