File: Schematics/flightcomputer2.kicad_sch (KiCad schematic)
At the start: 5 parts

Commit message: full output submited
Parts:
- R28, R29: LCSC (none) -> C17594
Changed lines of the file:
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@@
+			)
+		)
+		(property "LCSC" "C17594"
+			(at 181.61 68.58 90)
+			(hide yes)
+			(show_name no)
+			(do_not_autoplace no)
+			(effects
+				(font
+					(size 1.27 1.27)
+				)
 			)
 		)
@@
 			(hide yes)
 			(show_name no)
+			(do_not_autoplace no)
+			(effects
+				(font
+					(size 1.27 1.27)
+				)
+			)
+		)
+		(property "LCSC" "C17594"
+			(at 170.18 66.04 90)
+			(hide yes)
+			(show_name no)
